Commit message: replace cilinder with crazyflie mesh

File: crazyflie_ros2_description/urdf/crazyflie_description.urdf (robot description, URDF)
Before this commit: robot crazyflie, 1 links, 0 joints
Links:
- link crazyflie: geometry visual mesh filename=package://crazyflie_ros2_description/meshes/cf2_assembly.stl

Commit message: Added SLAM repo with slamtoolbox

File: crazyflie_ros2_description/urdf/crazyflie_description.urdf (robot description, URDF)
Before this commit: robot crazyflie, 1 links, 0 joints
Links:
- removed link crazyflie
- added link base_crazyflie; visual mesh filename=package://crazyflie_ros2_description/meshes/cf2_assembly.stl
